File: pcb/bedside-phone-control.kicad_pcb (KiCad board)
At the start: 2 copper layers, 49.1 x 32 mm, 28 parts, among them J1 USB_C_Receptacle_USB2.0_16P, J2 Conn_01x03, J3 USB_C_Receptacle_USB2.0_16P, J4 Conn_01x06, SW1 RotaryEncoder_Switch, SW3 EC12E2 424407, U1 ATmega328P-A, U2 MCP1703Ax-330xxDB, U3 MIC2026-1xM, U4 FUSB302B01MPX, Y1 16MHz

Commit message: getting there
Parts:
- moved R3 0.48 mm to (105.9, 46.4)
- moved R6 0.48 mm to (107.4, 46.4)
- moved R7 0.48 mm to (108.9, 46.4)
Connections:
- R3 pad 1: /D+ -> /D-
Routing:
- net /D-: track 23.3 -> 30.8 mm
- net /D+: track 20.5 -> 19.6 mm
Changed lines of the file:
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@@
   (setup
     (pad_to_mask_clearance 0)
+    (aux_axis_origin 73.025 67.31)
     (pcbplotparams
       (layerselection 0x00010fc_ffffffff)
@@
   )
   (footprint "Resistor_SMD:R_0603_1608Metric" (layer "F.Cu")
-    (at 108.458 46.355 -90)
+    (at 108.9406 46.355 -90)
     (descr "Resistor SMD 0603 (1608 Metric), square (rectangular) end terminal, IPC_7351 nominal, (Body size source: IPC-SM-782 page 72, https://www.pcb-3d.com/wordpress/wp-content/uploads/ipc-sm-782a_amendment_1_and_2.pdf), generated with kicad-footprint-generator")
     (tags "resistor")
@@
   )
   (footprint "Resistor_SMD:R_0603_1608Metric" (layer "F.Cu")
-    (at 105.41 46.355 -90)
+    (at 105.8926 46.355 -90)
     (descr "Resistor SMD 0603 (1608 Metric), square (rectangular) end terminal, IPC_7351 nominal, (Body size source: IPC-SM-782 page 72, https://www.pcb-3d.com/wordpress/wp-content/uploads/ipc-sm-782a_amendment_1_and_2.pdf), generated with kicad-footprint-generator")
     (tags "resistor")
@@
       (stroke (width 0.1) (type solid)) (layer "F.Fab"))
     (pad "1" smd roundrect (at -0.825 0 270) (size 0.8 0.95) (layers "F.Cu" "F.Paste" "F.Mask") (roundrect_rratio 0.25)
-      (net 13 "/D+") (pintype "passive"))
+      (net 14 "/D-") (pintype "passive"))
     (pad "2" smd roundrect (at 0.825 0 270) (size 0.8 0.95) (layers "F.Cu" "F.Paste" "F.Mask") (roundrect_rratio 0.25)
       (net 26 "/D+_PU") (pintype "passive"))
@@
   )
   (footprint "Resistor_SMD:R_0603_1608Metric" (layer "F.Cu")
-    (at 106.934 46.355 -90)
+    (at 107.4166 46.355 -90)
     (descr "Resistor SMD 0603 (1608 Metric), square (rectangular) end terminal, IPC_7351 nominal, (Body size source: IPC-SM-782 page 72, https://www.pcb-3d.com/wordpress/wp-content/uploads/ipc-sm-782a_amendment_1_and_2.pdf), generated with kicad-footprint-generator")
     (tags "resistor")
@@
   (segment (start 113.542 42.104) (end 114.292 42.854) (width 0.2) (layer "F.Cu") (net 13))
   (segment (start 104.521 46.863) (end 104.267 47.117) (width 0.2) (layer "F.Cu") (net 13))
-  (segment (start 105.41 45.53) (end 104.584 45.53) (width 0.2) (layer "F.Cu") (net 13))
   (segment (start 104.267 47.117) (end 102.933 47.117) (width 0.2) (layer "F.Cu") (net 13))
-  (segment (start 104.584 45.53) (end 104.521 45.593) (width 0.2) (layer "F.Cu") (net 13))
   (segment (start 112.960686 38.227) (end 113.942 39.208314) (width 0.2) (layer "F.Cu") (net 14))
+  (segment (start 102.233 47.6832) (end 102.4418 47.892) (width 0.2) (layer "F.Cu") (net 14))
   (segment (start 103.505 46.355) (end 104.121 46.355) (width 0.2) (layer "F.Cu") (net 14))
   (segment (start 114.042 40.459) (end 114.042 41.554) (width 0.2) (layer "F.Cu") (net 14))
   (segment (start 104.121 45.046315) (end 105.450314 43.717) (width 0.2) (layer "F.Cu") (net 14))
   (segment (start 111.126396 38.227) (end 112.960686 38.227) (width 0.2) (layer "F.Cu") (net 14))
+  (segment (start 102.233 46.166) (end 102.233 47.6832) (width 0.2) (layer "F.Cu") (net 14))
   (segment (start 113.942 39.208314) (end 113.942 39.959) (width 0.2) (layer "F.Cu") (net 14))
   (segment (start 102.933 45.783) (end 103.505 46.355) (width 0.2) (layer "F.Cu") (net 14))
@@
   (segment (start 106.276514 43.717) (end 107.775 42.218514) (width 0.2) (layer "F.Cu") (net 14))
   (segment (start 102.933 45.466) (end 102.933 45.783) (width 0.2) (layer "F.Cu") (net 14))
+  (segment (start 105.029 46.3936) (end 105.8926 45.53) (width 0.2) (layer "F.Cu") (net 14))
   (segment (start 113.942 39.959) (end 114.242 40.259) (width 0.2) (layer "F.Cu") (net 14))
   (segment (start 107.775 42.218514) (end 107.775 41.578396) (width 0.2) (layer "F.Cu") (net 14))
+  (segment (start 102.933 45.466) (end 102.233 46.166) (width 0.2) (layer "F.Cu") (net 14))
+  (segment (start 102.4418 47.892) (end 104.057686 47.892) (width 0.2) (layer "F.Cu") (net 14))
   (segment (start 105.450314 43.717) (end 106.276514 43.717) (width 0.2) (layer "F.Cu") (net 14))
+  (segment (start 104.057686 47.892) (end 105.029 46.920686) (width 0.2) (layer "F.Cu") (net 14))
   (segment (start 114.242 40.259) (end 114.042 40.459) (width 0.2) (layer "F.Cu") (net 14))
   (segment (start 107.775 41.578396) (end 111.126396 38.227) (width 0.2) (layer "F.Cu") (net 14))
   (segment (start 104.121 46.355) (end 104.121 45.046315) (width 0.2) (layer "F.Cu") (net 14))
+  (segment (start 105.029 46.920686) (end 105.029 46.3936) (width 0.2) (layer "F.Cu") (net 14))
   (via (at 113.538 43.471) (size 0.8) (drill 0.4) (layers "F.Cu" "B.Cu") (net 14))
   (via (at 114.242 40.259) (size 0.8) (drill 0.4) (layers "F.Cu" "B.Cu") (net 14))
@@
   (segment (start 82.28 42.839) (end 82.28 43.322) (width 0.25) (layer "F.Cu") (net 20))
   (segment (start 82.28 43.322) (end 80.39 45.212) (width 0.25) (layer "F.Cu") (net 20))
+  (segment (start 108.3316 44.615) (end 107.4166 45.53) (width 0.25) (layer "F.Cu") (net 21))
   (segment (start 117.336 44.057) (end 116.833 43.554) (width 0.25) (layer "F.Cu") (net 21))
+  (segment (start 110.46 45.53) (end 109.545 44.615) (width 0.25) (layer "F.Cu") (net 21))
   (segment (start 117.336 44.9655) (end 117.336 44.057) (width 0.25) (layer "F.Cu") (net 21))
-  (segment (start 107.849 44.615) (end 106.934 45.53) (width 0.25) (layer "F.Cu") (net 21))
+  (segment (start 109.545 44.615) (end 108.3316 44.615) (width 0.25) (layer "F.Cu") (net 21))
   (segment (start 110.46 45.53) (end 111.794 44.196) (width 0.25) (layer "F.Cu") (net 21))
-  (segment (start 110.46 45.53) (end 109.545 44.615) (width 0.25) (layer "F.Cu") (net 21))
   (segment (start 117.6095 44.9655) (end 117.336 44.9655) (width 0.25) (layer "F.Cu") (net 21))
   (segment (start 114.15 44.196) (end 114.792 43.554) (width 0.25) (layer "F.Cu") (net 21))
@@
   (segment (start 111.794 44.196) (end 114.15 44.196) (width 0.25) (layer "F.Cu") (net 21))
   (segment (start 117.8485 45.2045) (end 117.6095 44.9655) (width 0.25) (layer "F.Cu") (net 21))
-  (segment (start 109.545 44.615) (end 107.849 44.615) (width 0.25) (layer "F.Cu") (net 21))
   (segment (start 117.8485 45.728) (end 117.8485 45.2045) (width 0.25) (layer "F.Cu") (net 21))
   (segment (start 115.3235 45.27775) (end 115.3235 45.728) (width 0.25) (layer "F.Cu") (net 22))
   (segment (start 112.842 39.878) (end 113.042 40.078) (width 0.25) (layer "F.Cu") (net 22))
-  (segment (start 108.458 45.53) (end 109.256 46.328) (width 0.25) (layer "F.Cu") (net 22))
   (segment (start 114.091 45.728) (end 113.284 44.921) (width 0.25) (layer "F.Cu") (net 22))
-  (segment (start 109.256 46.328) (end 111.216 46.328) (width 0.25) (layer "F.Cu") (net 22))
+  (segment (start 108.9406 45.53) (end 109.7386 46.328) (width 0.25) (layer "F.Cu") (net 22))
   (segment (start 115.3235 45.728) (end 114.091 45.728) (width 0.25) (layer "F.Cu") (net 22))
+  (segment (start 111.216 46.328) (end 112.014 45.53) (width 0.25) (layer "F.Cu") (net 22))
+  (segment (start 109.7386 46.328) (end 111.216 46.328) (width 0.25) (layer "F.Cu") (net 22))
   (segment (start 115.836 44.9655) (end 115.63575 44.9655) (width 0.25) (layer "F.Cu") (net 22))
   (segment (start 115.63575 44.9655) (end 115.3235 45.27775) (width 0.25) (layer "F.Cu") (net 22))
-  (segment (start 111.216 46.328) (end 112.014 45.53) (width 0.25) (layer "F.Cu") (net 22))
   (segment (start 113.284 44.921) (end 112.675 45.53) (width 0.25) (layer "F.Cu") (net 22))
   (segment (start 113.042 40.078) (end 113.042 41.554) (width 0.25) (layer "F.Cu") (net 22))
@@
   (segment (start 96.647 49.022) (end 96.647 50.853) (width 0.2) (layer "F.Cu") (net 25))
   (segment (start 100.711 45.466) (end 100.203 45.974) (width 0.2) (layer "F.Cu") (net 25))
-  (segment (start 105.41 47.18) (end 105.41 48.08) (width 0.25) (layer "F.Cu") (net 26))
-  (segment (start 105.41 48.08) (end 103.892 49.598) (width 0.25) (layer "F.Cu") (net 26))
+  (segment (start 105.8926 47.5974) (end 103.892 49.598) (width 0.25) (layer "F.Cu") (net 26))
+  (segment (start 105.8926 47.18) (end 105.8926 47.5974) (width 0.25) (layer "F.Cu") (net 26))
   (segment (start 112.014 47.18) (end 110.46 47.18) (width 0.25) (layer "F.Cu") (net 28))
   (segment (start 106.902 51.848) (end 105.342 51.848) (width 0.25) (layer "F.Cu") (net 28))
   (segment (start 110.46 48.29) (end 106.902 51.848) (width 0.25) (layer "F.Cu") (net 28))
   (segment (start 110.46 47.18) (end 110.46 48.29) (width 0.25) (layer "F.Cu") (net 28))
-  (segment (start 108.458 47.18) (end 108.458 49.276) (width 0.25) (layer "F.Cu") (net 29))
-  (segment (start 108.458 47.18) (end 106.934 47.18) (width 0.25) (layer "F.Cu") (net 29))
-  (segment (start 108.458 49.276) (end 106.686 51.048) (width 0.25) (layer "F.Cu") (net 29))
+  (segment (start 108.9406 48.7934) (end 106.686 51.048) (width 0.25) (layer "F.Cu") (net 29))
+  (segment (start 108.9406 47.18) (end 108.9406 48.7934) (width 0.25) (layer "F.Cu") (net 29))
   (segment (start 106.686 51.048) (end 105.342 51.048) (width 0.25) (layer "F.Cu") (net 29))
+  (segment (start 108.9406 47.18) (end 107.4166 47.18) (width 0.25) (layer "F.Cu") (net 29))
   (segment (start 95.885 45.466) (end 96.393 45.974) (width 0.25) (layer "F.Cu") (net 30))
   (segment (start 93.726 45.466) (end 95.885 45.466) (width 0.25) (layer "F.Cu") (net 30))
@@
     (polygon
       (pts
-        (xy 72.644 35.306)
+        (xy 73.025 35.306)
         (xy 122.174 35.306)
         (xy 122.174 67.31)
-        (xy 72.644 67.056)
+        (xy 73.025 67.31)
       )
     )
