File: pcb/bedside-phone-control.kicad_sch (KiCad schematic)
At the start: 28 parts, among them J1 USB_C_Receptacle_USB2.0_16P, J2 Conn_01x03, J3 USB_C_Receptacle_USB2.0_16P, J4 Conn_01x06, SW1 RotaryEncoder_Switch, SW3 EC12E2 424407, U1 ATmega328P-A, U2 MCP1703Ax-330xxDB, U3 MIC2026-1xM, U4 FUSB302B01MPX, Y1 16MHz

Commit message: getting there
Connections:
- net D+: no longer R3.1
- net D-: now also R3.1
Other:
- title: (none) -> phonectl
Changed lines of the file:
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@@
 (kicad_sch (version 20230121) (generator eeschema)
   (paper "A4")
+  (title_block
+    (title "phonectl")
+    (date "2024-03-20")
+    (rev "2.0")
+  )
   (junction (at 191.77 60.96) (diameter 0) (color 0 0 0 0)
   )
-  (junction (at 189.23 138.43) (diameter 0) (color 0 0 0 0)
-  )
   (junction (at 190.5 88.9) (diameter 0) (color 0 0 0 0)
   )
@@
   )
   (junction (at 238.76 62.23) (diameter 0) (color 0 0 0 0)
+  )
+  (junction (at 189.23 140.97) (diameter 0) (color 0 0 0 0)
   )
   (junction (at 66.04 30.48) (diameter 0) (color 0 0 0 0)
@@
     (stroke (width 0) (type default))
   )
+  (wire (pts (xy 189.23 130.81) (xy 189.23 140.97))
+    (stroke (width 0) (type default))
+  )
   (wire (pts (xy 55.88 97.79) (xy 55.88 101.6))
     (stroke (width 0) (type default))
@@
     (stroke (width 0) (type default))
   )
-  (wire (pts (xy 189.23 138.43) (xy 185.42 138.43))
-    (stroke (width 0) (type default))
-  )
   (wire (pts (xy 52.07 35.56) (xy 63.5 35.56))
     (stroke (width 0) (type default))
@@
     (stroke (width 0) (type default))
   )
-  (wire (pts (xy 199.39 140.97) (xy 185.42 140.97))
+  (wire (pts (xy 199.39 140.97) (xy 189.23 140.97))
     (stroke (width 0) (type default))
   )
@@
     (stroke (width 0) (type default))
   )
-  (wire (pts (xy 189.23 130.81) (xy 189.23 138.43))
-    (stroke (width 0) (type default))
-  )
   (wire (pts (xy 190.5 106.68) (xy 190.5 109.22))
     (stroke (width 0) (type default))
@@
     (stroke (width 0) (type default))
   )
+  (wire (pts (xy 189.23 140.97) (xy 185.42 140.97))
+    (stroke (width 0) (type default))
+  )
   (wire (pts (xy 238.76 100.33) (xy 247.65 100.33))
     (stroke (width 0) (type default))
@@
     (stroke (width 0) (type default))
   )
-  (wire (pts (xy 199.39 138.43) (xy 189.23 138.43))
-    (stroke (width 0) (type default))
-  )
+  (wire (pts (xy 185.42 138.43) (xy 199.39 138.43))
+    (stroke (width 0) (type default))
+  )
